File: TheLightNing 2.0.kicad_pcb (KiCad board)
At the start: 2 copper layers, 80 x 60 mm, 31 parts, among them J1 motores izq, J2 motores der, J3 batt, J4 LED_izq, J5 dc jack, SW1 SW_SPDT, U1 L298(H)N, U2 ESP32_DEVKITC, U3 L7805, U4 L7805

Commit message: a
Parts:
- removed C6: 100uF 25v, EESTN5:CAP_ELEC_5x11mm
- removed D9: LED, EESTN5:Pin_strip_2
- removed R1: 330, EESTN5:RES0.3
- removed R2: 22 2W, EESTN5:RES0.3
- removed U4: L7805, EESTN5:TO-220
- added G***: LOGO, logo:yae, F.Cu at (144.6, 72.4)
- J1, J2: footprint EESTN5:JST-4V -> EESTN5:pin_strip_4
- J3: footprint EESTN5:BORNERA2_AZUL -> EESTN5:Pin_Header_2
- J5: value dc jack -> salida a modulo; footprint EESTN5:Pin_Strip_3 -> EESTN5:pin_strip_4
- moved J5 48.0 mm to (125.6, 81.8)
- moved J3 24.6 mm to (125.6, 88.9), turned to 0 degrees
- moved SW1 13.8 mm to (124.4, 85.6), turned to 180 degrees
- moved U3 11.2 mm to (124.2, 48.5), turned to 0 degrees
- moved C5 11.0 mm to (127.6, 60.5), turned to 90 degrees
- moved C4 7.93 mm to (126.7, 54.4), turned to -90 degrees
- moved C2 6.93 mm to (120.3, 60.7), turned to -90 degrees
- moved hole_2mm 5.00 mm to (117.5, 97.5)
- moved hole_2mm 5.00 mm to (117.5, 42.5)
- moved C3 2.02 mm to (121.6, 54.5), turned to -90 degrees
- moved J4 1.30 mm to (125.9, 75.0)
Connections:
- J3 pad 1: GND -> Net-(SW1-B)
- J3 pad 2: Net-(SW1-B) -> GND
- J5 pad 2: GND -> /Cargador
- J5 pad 3: Net-(J5-P3) -> +5V
Routing:
- net Net-(J5-P3): track 64.7 -> 0.00 mm
- net /Cargador: track 34.5 -> 3.80 mm
- net Net-(U4-OUT): track 16.7 -> 0.00 mm
- net Net-(SW1-B): track 17.6 -> 3.62 mm
- net VCC: track 172.8 -> 163.3 mm
- net +5V: track 160.7 -> 151.8 mm
- net Net-(D9-A): track 3.23 -> 0.00 mm
- net Net-(D7-A): track 66.6 -> 69.2 mm
- net Net-(D3-A): track 74.1 -> 75.6 mm
- net /led: track 8.98 -> 7.68 mm
- net Net-(D1-A): track 51.1 -> 52.3 mm
- net GND: vias 4 -> 3
Other:
- board size 80 x 60 mm -> 75 x 60 mm
- board text removed: "The LightNing 2.0"

Commit message: rework
Parts:
- removed G***: LOGO, logo:yae
- removed hole_2mm (x3): VAL**, EESTN5:hole_2mm
- moved D4 93.4 mm to (99.5, 87.4), turned to 0 degrees
- moved D2 86.9 mm to (99.5, 81.0), turned to 0 degrees
- moved D3 83.5 mm to (99.5, 90.6)
- moved J1 76.4 mm to (88.7, 86.8), turned to 90 degrees
- moved D1 75.5 mm to (99.5, 84.2)
- moved D6 61.4 mm to (139.7, 90.6)
- moved U1 58.0 mm to (110.7, 84.2), turned to 0 degrees
- moved D8 54.8 mm to (139.7, 84.2)
- moved D5 50.4 mm to (139.7, 87.4), turned to 0 degrees
- moved J5 43.8 mm to (98.3, 47.6)
- moved SW1 43.3 mm to (94.5, 54.2), turned to -90 degrees
- moved D7 42.8 mm to (139.7, 81.0), turned to 0 degrees
- moved J3 41.9 mm to (147.3, 53.0), turned to 90 degrees
- moved C3 39.1 mm to (89.5, 76.8), turned to 0 degrees
- moved C5 38.9 mm to (89.2, 54.2), turned to -90 degrees
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Connections:
- J1 pad 1: Net-(D7-A) -> Net-(D3-A)
- J1 pad 4: Net-(D7-A) -> Net-(D3-A)
- J2 pad 1: Net-(D3-A) -> Net-(D7-A)
- J2 pad 4: Net-(D3-A) -> Net-(D7-A)
- U2 pad 10: /IN4 -> unconnected-(U2-IO26-Pad10)
- U2 pad 11: /IN3 -> unconnected-(U2-IO27-Pad11)
- U2 pad 27: unconnected-(U2-IO16-Pad27) -> /IN1
- U2 pad 28: unconnected-(U2-IO17-Pad28) -> /IN2
- U2 pad 30: /buzz -> /IN3
- U2 pad 31: /led -> /IN4
- U2 pad 8: /IN1 -> /led
- U2 pad 9: /IN2 -> /buzz
Routing:
- net Net-(SW1-B): track 3.62 -> 53.2 mm
- net Net-(D3-A): track 75.6 -> 43.5 mm
- net Net-(D7-A): track 69.2 -> 42.3 mm
- net +5V: track 151.8 -> 125.5 mm, vias 1 -> 0
- net Net-(D5-A): track 60.7 -> 35.5 mm
- net VCC: track 163.3 -> 149.7 mm
- net Net-(D1-A): track 52.3 -> 41.6 mm
- net /led: track 7.68 -> 17.7 mm
- net /IN3: track 38.2 -> 28.5 mm
- net /IN4: track 33.7 -> 26.3 mm
- net /Cargador: track 3.80 -> 8.87 mm
- net /buzz: track 4.19 -> 7.40 mm
- net /IN2: track 12.1 -> 9.61 mm
- net /IN1: track 12.1 -> 9.64 mm
- net GND: vias 3 -> 0
Other:
- board size 75 x 60 mm -> 70 x 50 mm

Commit message: final version 1.5
Parts:
- removed BZ1: Buzzer, EESTN5:Pin_Header_2
- added J6: Sharp A, EESTN5:Pin_Strip_3, F.Cu at (150.1, 60.1)
- added J7: Sharp B, EESTN5:Pin_Strip_3, F.Cu at (150.1, 63.9)
- added J8: ampBuzz, EESTN5:Pin_Strip_3, F.Cu at (123.4, 47.6)
Connections:
- U2 pad 11: unconnected-(U2-IO27-Pad11) -> /sensor_a
- U2 pad 12: unconnected-(U2-IO14-Pad12) -> /sensor_b
- U2 pad 13: unconnected-(U2-IO12-Pad13) -> /sensor_c
Routing:
- net +5V: track 125.5 -> 214.6 mm
- net /sensor_b: track 0.00 -> 40.1 mm
- net /sensor_a: track 0.00 -> 34.3 mm
- net /buzz: track 7.40 -> 4.14 mm
