File: TheLightNing 2.0.kicad_sch (KiCad schematic)
At the start: 22 parts, among them J1 motores izq, J2 motores der, J3 batt, J4 LED_izq, SW1 SW_SPDT, U1 L298(H)N, U2 ESP32_DEVKITC, U3 L7805

Commit message: buzzer agregado
Parts:
- added BZ1: Buzzer, EESTN5:Pin_Header_2, symbol EESTN5:Buzzer
Connections:
- net GND: now also BZ1.2 (+)
- net buzz: now reaches U2.12 (IO14)
- net buzz: now also BZ1.1 (-)
Other:
- note added: "buzzer"
Changed lines of the file:
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@@
+    (stroke (width 0) (type default))
+  )
+  (wire (pts (xy 177.8 71.12) (xy 175.26 71.12))
     (stroke (width 0) (type default))
   )
@@
     (stroke (width 0) (type default))
   )
+  (polyline (pts (xy 163.83 82.55) (xy 203.2 82.55))
+    (stroke (width 0) (type default))
+  )
   (wire (pts (xy 166.37 49.53) (xy 175.26 49.53))
     (stroke (width 0) (type default))
@@
     (stroke (width 0) (type default))
   )
+  (wire (pts (xy 175.26 71.12) (xy 175.26 73.66))
+    (stroke (width 0) (type default))
+  )
   (wire (pts (xy 88.9 39.37) (xy 88.9 68.58))
     (stroke (width 0) (type default))
@@
     (stroke (width 0) (type default))
   )
+  (wire (pts (xy 175.26 66.04) (xy 177.8 66.04))
+    (stroke (width 0) (type default))
+  )
   (wire (pts (xy 58.42 96.52) (xy 55.88 96.52))
     (stroke (width 0) (type default))
@@
     (stroke (width 0) (type default))
   )
+  (polyline (pts (xy 203.2 82.55) (xy 203.2 55.88))
+    (stroke (width 0) (type default))
+  )
   (wire (pts (xy 191.77 39.37) (xy 191.77 36.83))
     (stroke (width 0) (type default))
@@
   )
   (wire (pts (xy 24.13 111.76) (xy 27.94 111.76))
+    (stroke (width 0) (type default))
+  )
+  (wire (pts (xy 24.13 124.46) (xy 27.94 124.46))
     (stroke (width 0) (type default))
   )
@@
     (effects (font (face "Arial Black") (size 4 4) (thickness 0.8) bold) (justify left bottom))
   )
+  (text "buzzer" (at 175.26 62.23 0)
+    (effects (font (face "Arial") (size 3 3) (thickness 0.6) bold) (justify left bottom))
+  )
   (text "DRIVER L298N" (at 54.61 25.4 0)
     (effects (font (face "Arial Black") (size 2.54 2.54) (thickness 0.508) bold) (justify left bottom))
@@
   )
   (label "IN3" (at 24.13 119.38 180) (fields_autoplaced)
+    (effects (font (size 1.27 1.27)) (justify right bottom))
+  )
+  (label "buzz" (at 24.13 124.46 180) (fields_autoplaced)
+    (effects (font (size 1.27 1.27)) (justify right bottom))
+  )
+  (label "buzz" (at 175.26 66.04 180) (fields_autoplaced)
     (effects (font (size 1.27 1.27)) (justify right bottom))
   )
@@
         (path "/e3664b64-e9fe-41a3-8f37-e0b2a1a8f77c"
           (reference "J1") (unit 1)
+        )
+      )
+    )
+  )
+  (symbol (lib_id "EESTN5:Buzzer") (at 180.34 68.58 0) (unit 1)
+    (in_bom yes) (on_board yes) (dnp no) (fields_autoplaced)
+    (property "Reference" "BZ1" (at 184.15 67.945 0)
+      (effects (font (size 1.27 1.27)) (justify left))
+    )
+    (property "Value" "Buzzer" (at 184.15 70.485 0)
+      (effects (font (size 1.27 1.27)) (justify left))
+    )
+    (property "Footprint" "EESTN5:Pin_Header_2" (at 179.705 66.04 90)
+      (effects (font (size 1.27 1.27)) hide)
+    )
+    (property "Datasheet" "" (at 179.705 66.04 90)
+      (effects (font (size 1.27 1.27)) hide)
+    )
+    (pin "1")
+    (pin "2")
+    (instances
+      (project "TheLightNing 2.0"
+        (path "/d8539005-a8e4-43a7-b9be-93452b210726"
+          (reference "BZ1") (unit 1)
         )
       )
@@
         )
       )
+    )
+  )
+  (symbol (lib_name "GND_1") (lib_id "power:GND") (at 175.26 73.66 0) (unit 1)
+    (in_bom yes) (on_board yes) (dnp no) (fields_autoplaced)
+    (property "Reference" "#PWR013" (at 175.26 80.01 0)
+      (effects (font (size 1.27 1.27)) hide)
+    )
+    (property "Value" "GND" (at 175.26 78.74 0)
+      (effects (font (size 1.27 1.27)))
+    )
+    (property "Footprint" "" (at 175.26 73.66 0)
+      (effects (font (size 1.27 1.27)) hide)
+    )
+    (property "Datasheet" "" (at 175.26 73.66 0)
+      (effects (font (size 1.27 1.27)) hide)
+    )
+    (pin "1")
+    (instances
+      (project "TheLightNing 2.0"
+        (path "/d8539005-a8e4-43a7-b9be-93452b210726"
+          (reference "#PWR013") (unit 1)
+        )
+      )

Commit message: re-made
Parts:
- removed H1: salida, EESTN5:hole_1mm, symbol Mechanical:MountingHole_Pad
- added C1: 100uF 25v, EESTN5:CAP_ELEC_5x11mm, symbol EESTN5:CAPAPOL
- added D1: LED, EESTN5:Pin_strip_2, symbol Device:LED
- added J5: dc jack, EESTN5:Pin_Strip_3, symbol EESTN5:Conn_01X03
- added R1: 330, EESTN5:RES0.3, symbol EESTN5:R
- added R2: 22 2W, EESTN5:RES0.3, symbol EESTN5:R
- added U1: L7805, EESTN5:TO-220, symbol Regulator_Linear:L7805
Connections:
- net GND: now also C1.2, J5.1 (P1), J5.2 (P2)
- net IN3: now also U2.11 (IO27); no longer U2.10 (IO26)
- net IN4: now also U2.10 (IO26); no longer U2.11 (IO27)
- net buzz: now also U2.30 (IO18); no longer U2.12 (IO14)
- net led: now also U2.31 (IO19); no longer U2.7 (IO32)
- net Cargador: now reaches SW1.1 (A)
- net Cargador: now also D1.1 (K), R2.2, U1.2 (GND)
- new net: C1.1, J5.3 (P3), U1.1 (IN)
- new net: R1.1, R2.1, U1.3 (OUT)
- new net: D1.2 (A), R1.2
Other:
- note added: "cargador"

Commit message: a
Parts:
- removed C1: 100uF 25v, EESTN5:CAP_ELEC_5x11mm, symbol EESTN5:CAPAPOL
- removed D1: LED, EESTN5:Pin_strip_2, symbol Device:LED
- removed J5: dc jack, EESTN5:Pin_Strip_3, symbol EESTN5:Conn_01X03
- removed R1: 330, EESTN5:RES0.3, symbol EESTN5:R
- removed R2: 22 2W, EESTN5:RES0.3, symbol EESTN5:R
- removed U1: L7805, EESTN5:TO-220, symbol Regulator_Linear:L7805
- added J5: salida a modulo, EESTN5:pin_strip_4, symbol Connector_Generic:Conn_01x04
- J1, J2: footprint EESTN5:JST-4V -> EESTN5:pin_strip_4
- J3: footprint EESTN5:BORNERA2_AZUL -> EESTN5:Pin_Header_2
Connections:
- net +5V: now also J5.3 (Pin_3)
- net Cargador: now also J5.2 (Pin_2)
- net GND: now also J3.2, J5.1 (Pin_1); no longer J3.1
- net VCC: now also J5.4 (Pin_4)
- net at SW1.2 (B): now also J3.1; no longer J3.2
Other:
- note added: "SALIDA A MODULO BATERIA"
- note removed: "cargador"

Commit message: rework
Connections:
- net IN1: now also U2.27 (IO16); no longer U2.8 (IO33)
- net IN2: now also U2.28 (IO17); no longer U2.9 (IO25)
- net IN3: now also U2.30 (IO18); no longer U2.11 (IO27)
- net IN4: now also U2.31 (IO19); no longer U2.10 (IO26)
- net buzz: now also U2.9 (IO25); no longer U2.30 (IO18)
- net led: now also U2.8 (IO33); no longer U2.31 (IO19)
- net at D7.1 (A), D8.2 (K), U1.13 (OUT3): now also J2.1 (Pin_1), J2.4 (Pin_4); no longer J1.1 (Pin_1), J1.4 (Pin_4)
- net at D3.1 (A), D4.2 (K), U1.2 (OUT1): now also J1.1 (Pin_1), J1.4 (Pin_4); no longer J2.1 (Pin_1), J2.4 (Pin_4)

Commit message: sharps
Parts:
- added J6: Sharp A, EESTN5:Pin_Strip_3, symbol Connector_Generic:Conn_01x03
- added J7: Sharp B, EESTN5:Pin_Strip_3, symbol Connector_Generic:Conn_01x03
- added J8: Sharp C, EESTN5:Pin_Strip_3, symbol Connector_Generic:Conn_01x03
Connections:
- net +5V: now also J6.2 (Pin_2), J7.2 (Pin_2), J8.2 (Pin_2)
- net GND: now also J6.3 (Pin_3), J7.3 (Pin_3), J8.3 (Pin_3)
- net sensor_a: now reaches U2.11 (IO27)
- net sensor_a: now also J6.1 (Pin_1)
- net sensor_b: now reaches U2.12 (IO14)
- net sensor_b: now also J7.1 (Pin_1)
- net sensor_c: now reaches U2.13 (IO12)
- net sensor_c: now also J8.1 (Pin_1)
Other:
- note added: "sensores SHARP"
- moved on the sheet: J5, U2

Commit message: final version 1.5
Parts:
- removed BZ1: Buzzer, EESTN5:Pin_Header_2, symbol EESTN5:Buzzer
- J8: value Sharp C -> ampBuzz
Connections:
- net +5V: now also J8.1 (Pin_1); no longer J8.2 (Pin_2)
- net buzz: now also J8.2 (Pin_2)
- net sensor_c: no longer J8.1 (Pin_1)
Other:
- moved on the sheet: J5
